File: eagle/5V-3.3VSupply_USB.sch (EAGLE design)
At the start: 27 parts, among them IC1 NJM2396, IC2 TA48M033F, IC3 LM358N, J1 DCIN, J2 5VOUT, J3 3V3OUT

Commit message: 基板図配置修正
Parts:
- added C8: 0.1uF, rcl:C-EU025-024X044
- LED1: value BLUE -> GREEN
- VR1: device v-reg:TL431CLP -> mylib2:TL431-INLINE
Connections:
- net GND: now also C8.2
- net N$1: now also C8.1
Changed lines of the file:
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@@
 <setting verticaltext="up"/>
 </settings>
-<grid distance="0.1" unitdist="inch" unit="inch" style="lines" multiple="1" display="yes" altdistance="0.01" altunitdist="inch" altunit="inch"/>
+<grid distance="0.1" unitdist="inch" unit="inch" style="lines" multiple="1" display="no" altdistance="0.01" altunitdist="inch" altunit="inch"/>
 <layers>
-<layer number="1" name="Top" color="4" fill="1" visible="yes" active="no"/>
-<layer number="16" name="Bottom" color="1" fill="1" visible="yes" active="no"/>
-<layer number="17" name="Pads" color="2" fill="1" visible="yes" active="no"/>
-<layer number="18" name="Vias" color="2" fill="1" visible="yes" active="no"/>
-<layer number="19" name="Unrouted" color="6" fill="1" visible="yes" active="no"/>
-<layer number="20" name="Dimension" color="15" fill="1" visible="yes" active="no"/>
-<layer number="21" name="tPlace" color="7" fill="1" visible="yes" active="no"/>
-<layer number="22" name="bPlace" color="7" fill="1" visible="yes" active="no"/>
-<layer number="23" name="tOrigins" color="15" fill="1" visible="yes" active="no"/>
-<layer number="24" name="bOrigins" color="15" fill="1" visible="yes" active="no"/>
-<layer number="25" name="tNames" color="7" fill="1" visible="yes" active="no"/>
-<layer number="26" name="bNames" color="7" fill="1" visible="yes" active="no"/>
-<layer number="27" name="tValues" color="7" fill="1" visible="yes" active="no"/>
-<layer number="28" name="bValues" color="7" fill="1" visible="yes" active="no"/>
+<layer number="1" name="Top" color="4" fill="1" visible="no" active="no"/>
+<layer number="16" name="Bottom" color="1" fill="1" visible="no" active="no"/>
+<layer number="17" name="Pads" color="2" fill="1" visible="no" active="no"/>
+<layer number="18" name="Vias" color="2" fill="1" visible="no" active="no"/>
+<layer number="19" name="Unrouted" color="6" fill="1" visible="no" active="no"/>
+<layer number="20" name="Dimension" color="15" fill="1" visible="no" active="no"/>
+<layer number="21" name="tPlace" color="7" fill="1" visible="no" active="no"/>
+<layer number="22" name="bPlace" color="7" fill="1" visible="no" active="no"/>
+<layer number="23" name="tOrigins" color="15" fill="1" visible="no" active="no"/>
+<layer number="24" name="bOrigins" color="15" fill="1" visible="no" active="no"/>
+<layer number="25" name="tNames" color="7" fill="1" visible="no" active="no"/>
+<layer number="26" name="bNames" color="7" fill="1" visible="no" active="no"/>
+<layer number="27" name="tValues" color="7" fill="1" visible="no" active="no"/>
+<layer number="28" name="bValues" color="7" fill="1" visible="no" active="no"/>
 <layer number="29" name="tStop" color="7" fill="3" visible="no" active="no"/>
 <layer number="30" name="bStop" color="7" fill="6" visible="no" active="no"/>
@@
 <layer number="35" name="tGlue" color="7" fill="4" visible="no" active="no"/>
 <layer number="36" name="bGlue" color="7" fill="5" visible="no" active="no"/>
-<layer number="37" name="tTest" color="7" fill="1" visible="yes" active="no"/>
-<layer number="38" name="bTest" color="7" fill="1" visible="yes" active="no"/>
+<layer number="37" name="tTest" color="7" fill="1" visible="no" active="no"/>
+<layer number="38" name="bTest" color="7" fill="1" visible="no" active="no"/>
 <layer number="39" name="tKeepout" color="4" fill="11" visible="no" active="no"/>
 <layer number="40" name="bKeepout" color="1" fill="11" visible="no" active="no"/>
@@
 <layer number="44" name="Drills" color="7" fill="1" visible="no" active="no"/>
 <layer number="45" name="Holes" color="7" fill="1" visible="no" active="no"/>
-<layer number="46" name="Milling" color="3" fill="1" visible="yes" active="no"/>
-<layer number="47" name="Measures" color="7" fill="1" visible="yes" active="no"/>
-<layer number="48" name="Document" color="7" fill="1" visible="yes" active="no"/>
-<layer number="49" name="Reference" color="7" fill="1" visible="yes" active="no"/>
-<layer number="50" name="dxf" color="7" fill="1" visible="yes" active="no"/>
-<layer number="51" name="tDocu" color="7" fill="1" visible="yes" active="no"/>
-<layer number="52" name="bDocu" color="7" fill="1" visible="yes" active="no"/>
+<layer number="46" name="Milling" color="3" fill="1" visible="no" active="no"/>
+<layer number="47" name="Measures" color="7" fill="1" visible="no" active="no"/>
+<layer number="48" name="Document" color="7" fill="1" visible="no" active="no"/>
+<layer number="49" name="Reference" color="7" fill="1" visible="no" active="no"/>
+<layer number="50" name="dxf" color="7" fill="1" visible="no" active="no"/>
+<layer number="51" name="tDocu" color="7" fill="1" visible="no" active="no"/>
+<layer number="52" name="bDocu" color="7" fill="1" visible="no" active="no"/>
 <layer number="90" name="Modules" color="5" fill="1" visible="yes" active="yes"/>
 <layer number="91" name="Nets" color="2" fill="1" visible="yes" active="yes"/>
@@
 <part name="C7" library="rcl" deviceset="CPOL-EU" device="E5-8.5" value="220uF"/>
 <part name="R1" library="rcl" deviceset="R-EU_" device="0207/7" value="1k"/>
-<part name="LED1" library="led" deviceset="LED" device="3MM" value="BLUE"/>
+<part name="LED1" library="led" deviceset="LED" device="3MM" value="GREEN"/>
 <part name="IC2" library="linear" deviceset="78*" device="TV" technology="05" value="TA48M033F"/>
 <part name="SUPPLY1" library="supply2" deviceset="GND" device=""/>
@@
 <part name="JP2" library="pinhead" deviceset="PINHD-1X2" device="" value="PWR SW"/>
 <part name="R2" library="rcl" deviceset="R-EU_" device="0207/7" value="200"/>
-<part name="VR1" library="v-reg" deviceset="TL431CLP" device="" value="TLE431"/>
+<part name="VR1" library="mylib2" deviceset="TL431-INLINE" device="" value="TLE431"/>
 <part name="R3" library="rcl" deviceset="R-EU_" device="0207/7" value="2.2k"/>
 <part name="R4" library="rcl" deviceset="R-EU_" device="0207/7" value="100k"/>
@@
 <part name="SUPPLY17" library="supply2" deviceset="GND" device=""/>
 <part name="SUPPLY18" library="supply2" deviceset="GND" device=""/>
+<part name="C8" library="rcl" deviceset="C-EU" device="025-024X044" value="0.1uF"/>
+<part name="SUPPLY19" library="supply2" deviceset="GND" device=""/>
 </parts>
 <sheets>
@@
 <instance part="JP2" gate="G$1" x="66.04" y="83.82" rot="R90"/>
 <instance part="R2" gate="G$1" x="147.32" y="116.84"/>
-<instance part="VR1" gate="G$1" x="66.04" y="114.3" rot="R90"/>
+<instance part="VR1" gate="G$1" x="66.04" y="111.76" rot="R90"/>
 <instance part="R3" gate="G$1" x="53.34" y="119.38"/>
 <instance part="R4" gate="G$1" x="60.96" y="142.24" rot="R180"/>
@@
 <instance part="SUPPLY17" gate="GND" x="134.62" y="134.62"/>
 <instance part="SUPPLY18" gate="GND" x="121.92" y="134.62"/>
+<instance part="C8" gate="G$1" x="144.78" y="160.02" rot="R90"/>
+<instance part="SUPPLY19" gate="GND" x="154.94" y="134.62"/>
 </instances>
 <busses>
@@
 <wire x1="129.54" y1="152.4" x2="121.92" y2="152.4" width="0.1524" layer="91"/>
 <wire x1="121.92" y1="152.4" x2="121.92" y2="137.16" width="0.1524" layer="91"/>
+</segment>
+<segment>
+<pinref part="C8" gate="G$1" pin="2"/>
+<pinref part="SUPPLY19" gate="GND" pin="GND"/>
+<wire x1="149.86" y1="160.02" x2="154.94" y2="160.02" width="0.1524" layer="91"/>
+<wire x1="154.94" y1="160.02" x2="154.94" y2="137.16" width="0.1524" layer="91"/>
 </segment>
 </net>
@@
 <pinref part="IC3" gate="P" pin="V+"/>
 <wire x1="134.62" y1="160.02" x2="134.62" y2="157.48" width="0.1524" layer="91"/>
+<pinref part="C8" gate="G$1" pin="1"/>
+<wire x1="142.24" y1="160.02" x2="134.62" y2="160.02" width="0.1524" layer="91"/>
+<junction x="134.62" y="160.02"/>
 </segment>
 </net>
@@
 </segment>
 </net>
-<net name="N$8" class="0">
-<segment>
-<pinref part="R3" gate="G$1" pin="2"/>
-<pinref part="IC3" gate="A" pin="-IN"/>
-<wire x1="58.42" y1="119.38" x2="60.96" y2="119.38" width="0.1524" layer="91"/>
-<pinref part="VR1" gate="G$1" pin="R"/>
-<wire x1="60.96" y1="119.38" x2="66.04" y2="119.38" width="0.1524" layer="91"/>
-<wire x1="66.04" y1="119.38" x2="71.12" y2="119.38" width="0.1524" layer="91"/>
-<wire x1="60.96" y1="116.84" x2="60.96" y2="119.38" width="0.1524" layer="91"/>
-<junction x="60.96" y="119.38"/>
-<pinref part="VR1" gate="G$1" pin="C"/>
-<wire x1="66.04" y1="116.84" x2="66.04" y2="119.38" width="0.1524" layer="91"/>
-<junction x="66.04" y="119.38"/>
-</segment>
-</net>
 <net name="N$9" class="0">
 <segment>
@@
 </segment>
 </net>
+<net name="N$8" class="0">
+<segment>
+<pinref part="R3" gate="G$1" pin="2"/>
+<pinref part="IC3" gate="A" pin="-IN"/>
+<wire x1="58.42" y1="119.38" x2="60.96" y2="119.38" width="0.1524" layer="91"/>
+<pinref part="VR1" gate="G$1" pin="C"/>
+<wire x1="60.96" y1="119.38" x2="66.04" y2="119.38" width="0.1524" layer="91"/>
+<wire x1="66.04" y1="119.38" x2="71.12" y2="119.38" width="0.1524" layer="91"/>
+<wire x1="66.04" y1="116.84" x2="66.04" y2="119.38" width="0.1524" layer="91"/>
+<junction x="66.04" y="119.38"/>
+<pinref part="VR1" gate="G$1" pin="R"/>
+<wire x1="60.96" y1="116.84" x2="60.96" y2="119.38" width="0.1524" layer="91"/>
+<junction x="60.96" y="119.38"/>
+</segment>
+</net>

Commit message: 基板図修正
Parts:
- R2: device rcl:R-EU_0207/7 -> rcl:R-EU_0207/2V
Changed lines of the file:
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@@
 <part name="J1" library="con-jack" deviceset="DCJ0303" device="" value="DCIN"/>
 <part name="JP2" library="pinhead" deviceset="PINHD-1X2" device="" value="PWR SW"/>
-<part name="R2" library="rcl" deviceset="R-EU_" device="0207/7" value="200"/>
+<part name="R2" library="rcl" deviceset="R-EU_" device="0207/2V" value="200"/>
 <part name="VR1" library="mylib2" deviceset="TL431-INLINE" device="" value="TLE431"/>
 <part name="R3" library="rcl" deviceset="R-EU_" device="0207/7" value="2.2k"/>

Commit message: コンパレーターの入力の正負を入れ替え
Connections:
- net N$8: now also IC3A.+IN; no longer IC3A.-IN
- net N$9: now also IC3A.-IN; no longer IC3A.+IN
Other:
- moved on the sheet: IC3A
Changed lines of the file:
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@@
 <instance part="R5" gate="G$1" x="76.2" y="142.24" rot="R180"/>
 <instance part="R6" gate="1" x="88.9" y="142.24" rot="R90"/>
-<instance part="IC3" gate="A" x="78.74" y="121.92"/>
+<instance part="IC3" gate="A" x="78.74" y="121.92" rot="MR180"/>
 <instance part="IC3" gate="B" x="137.16" y="149.86"/>
 <instance part="SUPPLY14" gate="GND" x="66.04" y="104.14"/>
@@
 <pinref part="R5" gate="G$1" pin="2"/>
 <wire x1="66.04" y1="142.24" x2="68.58" y2="142.24" width="0.1524" layer="91"/>
-<pinref part="IC3" gate="A" pin="+IN"/>
 <wire x1="68.58" y1="142.24" x2="71.12" y2="142.24" width="0.1524" layer="91"/>
-<wire x1="71.12" y1="124.46" x2="68.58" y2="124.46" width="0.1524" layer="91"/>
 <wire x1="68.58" y1="124.46" x2="68.58" y2="142.24" width="0.1524" layer="91"/>
 <junction x="68.58" y="142.24"/>
+<pinref part="IC3" gate="A" pin="-IN"/>
+<wire x1="71.12" y1="124.46" x2="68.58" y2="124.46" width="0.1524" layer="91"/>
 </segment>
 </net>
@@
 <segment>
 <pinref part="R3" gate="G$1" pin="2"/>
-<pinref part="IC3" gate="A" pin="-IN"/>
 <wire x1="58.42" y1="119.38" x2="60.96" y2="119.38" width="0.1524" layer="91"/>
 <pinref part="VR1" gate="G$1" pin="C"/>
 <wire x1="60.96" y1="119.38" x2="66.04" y2="119.38" width="0.1524" layer="91"/>
-<wire x1="66.04" y1="119.38" x2="71.12" y2="119.38" width="0.1524" layer="91"/>
 <wire x1="66.04" y1="116.84" x2="66.04" y2="119.38" width="0.1524" layer="91"/>
-<junction x="66.04" y="119.38"/>
 <pinref part="VR1" gate="G$1" pin="R"/>
 <wire x1="60.96" y1="116.84" x2="60.96" y2="119.38" width="0.1524" layer="91"/>
 <junction x="60.96" y="119.38"/>
-</segment>
-</net>
+<pinref part="IC3" gate="A" pin="+IN"/>
+<wire x1="71.12" y1="119.38" x2="66.04" y2="119.38" width="0.1524" layer="91"/>
+<junction x="66.04" y="119.38"/>
+</segment>
+</net>
